Commit message: first commit

File: e05/urdf/e05.urdf (robot description, URDF)
Before this commit: robot e05, 8 links, 7 joints
Joints:
- joint joint5: limit lower=-3.14 upper=3.14 effort=100 velocity=3 -> lower=-3.14 upper=-1.5 effort=100 velocity=3

File: e05/urdf/e05_mujoco.urdf (robot description, URDF)
Before this commit: robot e05, 18 links, 17 joints
Joints:
- joint gripper_finger1_joint: limit lower=0.0 upper=0.804 effort=1000 velocity=2.0 -> lower=0.0 upper=0.378 effort=1000 velocity=2.0

File: robotiq/robotiq_85_gripper/robotiq_85_description/urdf/robotiq_85_gripper.urdf.xacro (robot description, xacro)
@@ -39,5 +39,5 @@
             <axis xyz="0 0 1"/>
             <origin rpy="${pi} 0.0 0.0" xyz="0.05490451627 0.03060114443 0.0"/>
-            <limit lower="0.0" upper="0.804" velocity="2.0" effort="1000"/>
+            <limit lower="0.0" upper="0.378" velocity="2.0" effort="1000"/>
         </joint>
         <joint name="${prefix}gripper_finger2_joint" type="revolute">

Commit message: fix unused joints

File: e05/urdf/e05.urdf (robot description, URDF)
Before this commit: robot e05, 8 links, 7 joints
Joints:
- removed joint joint1
- removed joint joint2
- removed joint joint3
- removed joint joint4
- removed joint joint5
- removed joint joint6
- added joint joint_0: type revolute, parent base_link, child link1, origin xyz=0 0 0.0735 rpy=0 0 1.5707963267949, axis 0 0 1, limit lower=0 upper=0 effort=100 velocity=3
- added joint joint_1: type revolute, parent link1, child link2, origin xyz=0 0 0.146499999728183 rpy=-1.5707963267949 0 1.5707963267949, axis 0 0 -1, limit lower=0 upper=0 effort=100 velocity=3
- added joint joint_2: type revolute, parent link2, child link3, origin xyz=0 -0.38 0 rpy=0 0 0, axis 0 0 -1, limit lower=0 upper=0 effort=100 velocity=3
- added joint joint_3: type revolute, parent link3, child link4, origin xyz=0 0 0 rpy=-1.5707963267949 0 -1.57079632679489, axis 0 0 1, limit lower=0 upper=0 effort=100 velocity=3
- added joint joint_4: type revolute, parent link4, child link5, origin xyz=0 0 -0.42 rpy=-1.5708 1.5708 0, axis 0 0 1, limit lower=-3.14 upper=-1.5 effort=100 velocity=3
- added joint joint_5: type revolute, parent link5, child link6, origin xyz=0 0.155 0 rpy=-1.5708 0 0, axis 0 0 -1, limit lower=0 upper=0 effort=100 velocity=3

File: e05/urdf/e05.xacro (robot description, xacro)
@@ -21,10 +21,10 @@
    </xacro:macro>
     <!-- Transmissions for ros control -->
-    <xacro:transmission_block joint_name="joint1"/>
-    <xacro:transmission_block joint_name="joint2"/>
-    <xacro:transmission_block joint_name="joint3"/>
-    <xacro:transmission_block joint_name="joint4"/>
-    <xacro:transmission_block joint_name="joint5"/>
-    <xacro:transmission_block joint_name="joint6"/>
+    <xacro:transmission_block joint_name="joint_0"/>
+    <xacro:transmission_block joint_name="joint_1"/>
+    <xacro:transmission_block joint_name="joint_2"/>
+    <xacro:transmission_block joint_name="joint_3"/>
+    <xacro:transmission_block joint_name="joint_4"/>
+    <xacro:transmission_block joint_name="joint_5"/>
     <!-- <xacro:include filename="$(find e05)/urdf/e05.gazebo.xacro" /> -->
     <!-- 机器人固定在世界坐标系下 -->

File: e05/urdf/e05_mujoco.urdf (robot description, URDF)
Before this commit: robot e05, 18 links, 17 joints
Joints:
- removed joint joint1
- removed joint joint2
- removed joint joint3
- removed joint joint4
- removed joint joint5
- removed joint joint6
- added joint joint_0: type revolute, parent base_link, child link1, origin xyz=0 0 0.0735 rpy=0 0 0, axis 0 0 1, limit lower=-3.14 upper=3.14 effort=100 velocity=3
- added joint joint_1: type revolute, parent link1, child link2, origin xyz=0 0 0.146499999728183 rpy=-1.5707963267949 0 1.5707963267949, axis 0 0 -1, limit lower=-3.14 upper=3.14 effort=100 velocity=3
- added joint joint_2: type revolute, parent link2, child link3, origin xyz=0 -0.38 0 rpy=0 0 1.57079632679489, axis 0 0 -1, limit lower=-3.14 upper=3.14 effort=100 velocity=3
- added joint joint_3: type revolute, parent link3, child link4, origin xyz=0 0 0 rpy=-1.5707963267949 0 -1.57079632679489, axis 0 0 1, limit lower=-3.14 upper=3.14 effort=100 velocity=3
- added joint joint_4: type revolute, parent link4, child link5, origin xyz=0 0 -0.42 rpy=-1.5708 0 0, axis 0 0 1, limit lower=-3.14 upper=3.14 effort=100 velocity=3
- added joint joint_5: type revolute, parent link5, child link6, origin xyz=0 0.155 0 rpy=-1.5708 0 0, axis 0 0 -1, limit lower=-3.14 upper=3.14 effort=100 velocity=3

File: e05/urdf/e05_mujoco.xacro (robot description, xacro)
@@ -27,10 +27,10 @@
    </xacro:macro>
     <!-- Transmissions for ros control -->
-    <xacro:transmission_block joint_name="joint1"/>
-    <xacro:transmission_block joint_name="joint2"/>
-    <xacro:transmission_block joint_name="joint3"/>
-    <xacro:transmission_block joint_name="joint4"/>
-    <xacro:transmission_block joint_name="joint5"/>
-    <xacro:transmission_block joint_name="joint6"/>
+    <xacro:transmission_block joint_name="joint_0"/>
+    <xacro:transmission_block joint_name="joint_1"/>
+    <xacro:transmission_block joint_name="joint_2"/>
+    <xacro:transmission_block joint_name="joint_3"/>
+    <xacro:transmission_block joint_name="joint_4"/>
+    <xacro:transmission_block joint_name="joint_5"/>
     <!-- <xacro:include filename="$(find e05)/urdf/e05.gazebo.xacro" /> -->
     <!-- 机器人固定在世界坐标系下 -->
